File: 8RelaySwitch.sch (EAGLE design)
At the start: 60 parts, among them IC1 LNK304, IC3 MC33269ST-3.3T3, K1 FRS1B, K11 FRS1B, K12 FRS1B, K13 FRS1B, K14 FRS1B, K15 FRS1B, K16 FRS1B, K2 FRS1B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

Commit message: aaa
aaa
Parts:
- added C1, C2: 100nF, resistor:C-EUC2012
- added R16: 1 K, resistor:R-EU_M2012
- added U$3: ESP03, RemoteHome:ESP03
- JP1: value (none) -> PINHD1X5SQUARE; device pinhead-2:PINHD-1X05_2.54-S -> eagle-library-edeca.net-v5:PINHD1X5SQUARE
- L1: device inductor-neosid:BS11 -> inductor-neosid:SD8
- R14: value 470 -> 1K
- R15: value 470 -> 1 K
Connections:
- net N$10 renamed S
- new net N$10: R15.1, U$3.TX
- new net N$12: R16.1, U$3.RX
- net 5V1: now also C2.2
- net D0_RX: now also R15.2
- net D1_TX: now also R16.2
- net D2: now also U$3.EN
- net D9: no longer R14.1, R15.2
- net GND: now also C1.1, C2.1, R14.1, U$3.GND, U$3.GPIO15; no longer R15.1
- net VCC: now also C1.2, U$3.VDD
Other:
- moved on the sheet: C10, C11, C5, C9, R14, R15
