File: ChangeOverSwitch.brd (EAGLE design)
At the start: 28.9 x 37.5 mm, 36 parts, among them IC3 MC33269ST-3.3T3, K1 FRS1B, T1 BC846, X1 16 MHz

Commit message: aaa
aaa
Parts:
- removed JP2: (no value), pinhead-2:1X05M
- removed R14: 560, resistor:M2012
- removed R3, R7: 10K, resistor:M2012
- removed R5: 20K, resistor:M2012
- removed X2: (no value), con-ptr500:AK500/5
- added C3, C4: 0.1, resistor:C2012
- added X3: (no value), con-ptr500:AK500/5
- INTERFACE: value (none) -> PINHD1X5SQUARE; device pinhead-2:1X05-S -> eagle-library-edeca.net-v5:PINHD1X05-SQUARE
- R4: value 470 -> 1K
- moved C10 15.0 mm to (8.41, 35.1)
- moved R4 15.0 mm to (14.3, 25.9), turned to 270 degrees
- moved C7 10.5 mm to (26.5, 14.4), turned to 180 degrees
- moved D3 7.36 mm to (14.0, 21.9), turned to 0 degrees
- moved R13 6.48 mm to (21.2, 18.8), turned to 90 degrees
- moved R12 6.21 mm to (21.2, 14.8), turned to 90 degrees
- moved D4 5.68 mm to (15.4, 17.0)
- moved C9 5.57 mm to (7.57, 11.5), turned to 0 degrees
- moved C1 5.47 mm to (13.7, 8.72), turned to 270 degrees
- moved L1 5.43 mm to (13.7, 11.6), turned to 180 degrees
- moved C5 3.90 mm to (5.33, 20.4), turned to 270 degrees
- moved R2 3.38 mm to (13.7, 30.6), turned to 180 degrees
- moved R10 2.93 mm to (22.8, 25.4), turned to 180 degrees
- moved R1 2.74 mm to (2.22, 21.1)
- moved LNK 2.39 mm to (25.6, 18.1)
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Connections:
- net N$10 renamed S
- removed net N$11: K1.S, X2.3
- removed net N$12: K1.O, X2.5
- new net N$10: K1.P@, X3.4
- new net N$6: K1.O, X3.5
- net 5V: now also C3.1; no longer JP2.1
- net A0: no longer JP2.4, R5.2
- net A1: no longer JP2.5, R7.2
- net D3: no longer JP2.2, R3.2
- net D9: no longer R14.2, R4.1
- net GND: now also C3.2, C4.2, R4.1; no longer JP2.3, R14.1, R3.1, R5.1, R7.1
- net N$7: now also K1.S, X3.3; no longer R11.1, X2.1
- net N$8: now also R11.1, X3.1; no longer K1.P@, X2.4
- net N$9: now also X3.2; no longer X2.2
- net VCC: now also C4.1
Routing:
- net GND: track 66.9 -> 14.5 mm, vias 11 -> 13
- net D9: track 39.1 -> 0.00 mm, vias 2 -> 0
- net 5V: track 72.6 -> 35.9 mm, vias 2 -> 0
- net A1: track 35.9 -> 0.00 mm, vias 3 -> 0
- net D3: track 33.7 -> 0.00 mm, vias 1 -> 0
- net S: track 56.7 -> 27.7 mm
- net A0: track 28.7 -> 0.00 mm, vias 4 -> 0
- net N$10: track 0.00 -> 21.6 mm
- net N$5: track 76.8 -> 59.3 mm
- net N$8: track 20.8 -> 5.86 mm
- net FB: track 19.4 -> 4.60 mm, vias 2 -> 0
- net N$2: track 8.05 -> 17.2 mm
- net RST: track 52.6 -> 43.8 mm, vias 5 -> 2
- net N$11: track 6.99 -> 0.00 mm
- net N$12: track 6.12 -> 0.00 mm
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- added copper zone on layer 1, net S
- added copper zone on layer 16, net S
