File: ChangeOverSwitch.sch (EAGLE design)
At the start: 36 parts, among them IC3 MC33269ST-3.3T3, K1 FRS1B, T1 BC846, X1 16 MHz

Commit message: aaa
aaa
Parts:
- removed JP2: (no value), pinhead-2:PINHD-1X05_2.00
- removed R14: 560, resistor:R-EU_M2012
- removed R3, R7: 10K, resistor:R-EU_M2012
- removed R5: 20K, resistor:R-EU_M2012
- removed X2: (no value), con-ptr500:AK500/5
- added C3, C4: 0.1, resistor:C-EUC2012
- added X3: (no value), con-ptr500:AK500/5
- INTERFACE: value (none) -> PINHD1X5SQUARE; device pinhead-2:PINHD-1X05_2.54-S -> eagle-library-edeca.net-v5:PINHD1X5SQUARE
- R4: value 470 -> 1K
Connections:
- net N$10 renamed S
- removed net N$11: K12.S, X2-3.KL
- removed net N$12: K12.O, X2-5.KL
- new net N$10: K12.P@1, X3-4.KL
- new net N$6: K12.O, X3-5.KL
- net 5V: now also C3.1; no longer JP2.1
- net A0: no longer JP2.4, R5.2
- net A1: no longer JP2.5, R7.2
- net D3: no longer JP2.2, R3.2
- net D9: no longer R14.2, R4.1
- net GND: now also C3.2, C4.2, R4.1; no longer JP2.3, R14.1, R3.1, R5.1, R7.1
- net N$7: now also K12.S, X3-3.KL; no longer R11.1, X2-1.KL
- net N$8: now also R11.1, X3-1.KL; no longer K12.P@1, X2-4.KL
- net N$9: now also X3-2.KL; no longer X2-2.KL
- net VCC: now also C4.1
Other:
- moved on the sheet: C1, C5
