File: DoubleSwitch.sch (EAGLE design)
At the start: 36 parts, among them IC1 LNK304, IC3 MC33269ST-3.3T3, K1 FRS1B, K2 FRS1B, T1 BC846, T2 BC846, X1 16 MHz

Commit message: aaa
aaa
Parts:
- removed R14: 560, resistor:R-EU_M2012
- added C2, C3: 0.1, resistor:C-EUC2012
- JP1: value (none) -> PINHD1X5SQUARE; device pinhead-2:PINHD-1X05_2.54-S -> eagle-library-edeca.net-v5:PINHD1X5SQUARE
- R4: value 560 -> 1K
Connections:
- net N$10 renamed S
- removed net N$8: K12.P, K22.P, R11.1, X2-4.KL
- net 5V: now also C2.1
- net D9: no longer R14.2, R4.1
- net GND: now also C2.2, C3.2, R4.1; no longer R14.1
- net N$16: now also K12.P, R11.1, X2-4.KL
- net VCC: now also C3.1
Other:
- moved on the sheet: C5
