File: sensorAA.brd (EAGLE design)
At the start: 29.3 x 16.2 mm, 21 parts, among them IC1 LM75AD, IC4 RFM69, X1 16 MHz

Commit message: aaa
aaa
Parts:
- removed R4: 10k, resistor:R2012
- INTERFACE: value (none) -> PINHD1X5SQUARE; device pinhead-2:1X05-S -> eagle-library-edeca.net-v5:PINHD1X05-SQUARE
- moved GND 0.54 mm to (7.09, 1.42)
Connections:
- net D3: no longer R4.2
- net D4: now also JP1.3
- net D5: now also R5.1
- net GND: no longer R4.1, R5.1
- net VCC: no longer JP1.3
Routing:
- net D5: track 0.00 -> 6.94 mm
- net D4: track 0.00 -> 6.18 mm
- net GND: track 52.7 -> 48.6 mm, vias 18 -> 17
- net D3: track 25.6 -> 21.9 mm
- net VCC: track 77.2 -> 78.3 mm
