File: sensorAA.sch (EAGLE design)
At the start: 21 parts, among them IC1 LM75AD, IC4 RFM69, X1 16 MHz

Commit message: aaa
aaa
Parts:
- removed R4: 10k, resistor:R-EU_R2012
- INTERFACE: value (none) -> PINHD1X5SQUARE; device pinhead-2:PINHD-1X05_2.54-S -> eagle-library-edeca.net-v5:PINHD1X5SQUARE
Connections:
- net D3: no longer R4.2
- net D4: now also JP1.3
- net D5: now also R5.1
- net GND: no longer R4.1, R5.1
- net VCC: no longer JP1.3
Changed lines of the file:
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@@
 <part name="C5" library="resistor" deviceset="C-EU" device="C2012" value="0.1"/>
 <part name="R1" library="resistor" deviceset="R-EU_" device="R2012" value="10k"/>
-<part name="INTERFACE" library="pinhead-2" deviceset="PINHD-1X05" device="_2.54-S"/>
+<part name="INTERFACE" library="eagle-library-edeca.net-v5" deviceset="PINHD1X5" device="SQUARE"/>
 <part name="P+2" library="SparkFun" deviceset="VCC" device="" value="3.3V"/>
 <part name="SUPPLY7" library="supply2" deviceset="GND" device=""/>
@@
 <part name="SUPPLY8" library="supply2" deviceset="GND" device=""/>
 <part name="SUPPLY9" library="supply2" deviceset="GND" device=""/>
-<part name="SUPPLY10" library="SparkFun" deviceset="VCC" device="" value="3.3V"/>
 <part name="R2" library="resistor" deviceset="R-EU_" device="R2012" value="10k"/>
 <part name="R3" library="resistor" deviceset="R-EU_" device="R2012" value="10k"/>
 <part name="SUPPLY11" library="SparkFun" deviceset="VCC" device="" value="3.3V"/>
-<part name="R4" library="resistor" deviceset="R-EU_" device="R2012" value="10k"/>
 <part name="U$2" library="RemoteHome" deviceset="AVRHEADER" device="" technology="DIP"/>
 <part name="RESET" library="switch-tact" deviceset="DTSM-3" device="" value=""/>
 <part name="SUPPLY12" library="supply2" deviceset="GND" device=""/>
 <part name="R5" library="resistor" deviceset="R-EU_" device="R2012" value="10k"/>
-<part name="SUPPLY13" library="supply2" deviceset="GND" device=""/>
 <part name="JP1" library="pinhead-2" deviceset="PINHD-1X04" device="_2.54-S"/>
 <part name="JP2" library="pinhead-2" deviceset="PINHD-1X01" device="_2.54"/>
@@
 <instance part="C5" gate="G$1" x="-5.08" y="119.38"/>
 <instance part="R1" gate="G$1" x="0" y="137.16"/>
-<instance part="INTERFACE" gate="A" x="87.63" y="114.3"/>
+<instance part="INTERFACE" gate="G$1" x="87.63" y="114.3"/>
 <instance part="P+2" gate="1" x="76.2" y="120.65"/>
 <instance part="SUPPLY7" gate="GND" x="30.48" y="22.86"/>
@@
 <instance part="SUPPLY8" gate="GND" x="144.78" y="109.22"/>
 <instance part="SUPPLY9" gate="GND" x="121.92" y="76.2"/>
-<instance part="SUPPLY10" gate="1" x="121.92" y="101.6"/>
 <instance part="R2" gate="G$1" x="111.76" y="134.62" rot="R90"/>
 <instance part="R3" gate="G$1" x="101.6" y="132.08" rot="R90"/>
 <instance part="SUPPLY11" gate="1" x="106.68" y="139.7"/>
-<instance part="R4" gate="G$1" x="116.84" y="83.82" rot="R90"/>
 <instance part="U$2" gate="G$1" x="175.26" y="132.08"/>
 <instance part="RESET" gate="G$1" x="12.7" y="147.32" rot="R270"/>
 <instance part="SUPPLY12" gate="GND" x="17.78" y="144.78"/>
 <instance part="R5" gate="G$1" x="81.28" y="144.78" rot="R90"/>
-<instance part="SUPPLY13" gate="GND" x="81.28" y="137.16"/>
 <instance part="JP1" gate="A" x="127" y="91.44" rot="R180"/>
 <instance part="JP2" gate="A" x="83.82" y="154.94"/>
@@
 </segment>
 <segment>
-<pinref part="INTERFACE" gate="A" pin="5"/>
+<pinref part="INTERFACE" gate="G$1" pin="5"/>
 <pinref part="SUPPLY3" gate="GND" pin="GND"/>
-<wire x1="85.09" y1="109.22" x2="76.2" y2="109.22" width="0.1524" layer="91"/>
+<wire x1="87.63" y1="109.22" x2="76.2" y2="109.22" width="0.1524" layer="91"/>
 <wire x1="76.2" y1="109.22" x2="76.2" y2="107.95" width="0.1524" layer="91"/>
 </segment>
@@
 <wire x1="121.92" y1="86.36" x2="121.92" y2="78.74" width="0.1524" layer="91"/>
 <pinref part="SUPPLY9" gate="GND" pin="GND"/>
-<pinref part="R4" gate="G$1" pin="1"/>
-<wire x1="116.84" y1="78.74" x2="121.92" y2="78.74" width="0.1524" layer="91"/>
-<junction x="121.92" y="78.74"/>
 <pinref part="JP1" gate="A" pin="1"/>
 </segment>
@@
 <pinref part="RESET" gate="G$1" pin="2"/>
 <pinref part="SUPPLY12" gate="GND" pin="GND"/>
-</segment>
-<segment>
-<pinref part="R5" gate="G$1" pin="1"/>
-<pinref part="SUPPLY13" gate="GND" pin="GND"/>
 </segment>
 </net>
@@
 </segment>
 <segment>
-<pinref part="INTERFACE" gate="A" pin="1"/>
-<wire x1="85.09" y1="119.38" x2="76.2" y2="119.38" width="0.1524" layer="91"/>
+<pinref part="INTERFACE" gate="G$1" pin="1"/>
+<wire x1="87.63" y1="119.38" x2="76.2" y2="119.38" width="0.1524" layer="91"/>
 <wire x1="76.2" y1="119.38" x2="76.2" y2="120.65" width="0.1524" layer="91"/>
 <pinref part="P+2" gate="1" pin="VCC"/>
@@
 <wire x1="30.48" y1="54.61" x2="30.48" y2="53.34" width="0.1524" layer="91"/>
 <pinref part="IC4" gate="G$1" pin="VCC"/>
-</segment>
-<segment>
-<wire x1="129.54" y1="91.44" x2="121.92" y2="91.44" width="0.1524" layer="91"/>
-<pinref part="SUPPLY10" gate="1" pin="VCC"/>
-<wire x1="121.92" y1="91.44" x2="121.92" y2="101.6" width="0.1524" layer="91"/>
-<pinref part="JP1" gate="A" pin="3"/>
 </segment>
 <segment>
@@
 <wire x1="55.88" y1="101.6" x2="68.58" y2="101.6" width="0.1524" layer="91"/>
 </segment>
+<segment>
+<pinref part="R5" gate="G$1" pin="1"/>
+<wire x1="81.28" y1="139.7" x2="91.44" y2="139.7" width="0.1524" layer="91"/>
+<label x="91.44" y="139.7" size="1.778" layer="95"/>
+</segment>
 </net>
 <net name="D4" class="0">
@@
 <pinref part="ATMEGA328" gate="G$1" pin="PD4(XCK/T0)"/>
 </segment>
+<segment>
+<wire x1="129.54" y1="91.44" x2="121.92" y2="91.44" width="0.1524" layer="91"/>
+<wire x1="121.92" y1="91.44" x2="121.92" y2="101.6" width="0.1524" layer="91"/>
+<pinref part="JP1" gate="A" pin="3"/>
+<label x="121.92" y="101.6" size="1.778" layer="95"/>
+</segment>
 </net>
 <net name="D3" class="0">
@@
 </segment>
 <segment>
-<wire x1="129.54" y1="88.9" x2="116.84" y2="88.9" width="0.1524" layer="91"/>
-<pinref part="R4" gate="G$1" pin="2"/>
-<wire x1="116.84" y1="88.9" x2="111.76" y2="88.9" width="0.1524" layer="91"/>
-<junction x="116.84" y="88.9"/>
+<wire x1="129.54" y1="88.9" x2="111.76" y2="88.9" width="0.1524" layer="91"/>
 <pinref part="JP1" gate="A" pin="2"/>
 <label x="109.22" y="88.9" size="1.778" layer="95"/>
@@
 <label x="58.42" y="111.76" size="1.778" layer="95"/>
 <pinref part="ATMEGA328" gate="G$1" pin="PD1(TXD)"/>
-<wire x1="55.88" y1="111.76" x2="85.09" y2="111.76" width="0.1524" layer="91"/>
-<pinref part="INTERFACE" gate="A" pin="4"/>
+<wire x1="55.88" y1="111.76" x2="87.63" y2="111.76" width="0.1524" layer="91"/>
+<pinref part="INTERFACE" gate="G$1" pin="4"/>
 </segment>
 </net>
@@
 <label x="58.42" y="114.3" size="1.778" layer="95"/>
 <pinref part="ATMEGA328" gate="G$1" pin="PD0(RXD)"/>
-<wire x1="55.88" y1="114.3" x2="85.09" y2="114.3" width="0.1524" layer="91"/>
-<pinref part="INTERFACE" gate="A" pin="3"/>
-</segment>
-</net>
+<wire x1="55.88" y1="114.3" x2="87.63" y2="114.3" width="0.1524" layer="91"/>
+<pinref part="INTERFACE" gate="G$1" pin="3"/>
+</segment>
+</net>
