File: SimpleSwitch.sch (EAGLE design)
At the start: 36 parts, among them IC3 MC33269ST-3.3T3, K1 FRS1B, T1 BC846, X1 16 MHz

Commit message: aaa
aaa
Parts:
- removed JP2: (no value), pinhead-2:PINHD-1X05_2.00
- removed R14: 560, resistor:R-EU_M2012
- removed R3: 10K, resistor:R-EU_M2012
- removed R5: 20K, resistor:R-EU_M2012
- added C3, C4: 0.1, resistor:C-EUC2012
- added R6: 1 K, resistor:R-EU_M2012
- added U$5: ESP03, RemoteHome:ESP03
- INTERFACE: value (none) -> PINHD1X5SQUARE; device pinhead-2:PINHD-1X05_2.54-S -> eagle-library-edeca.net-v5:PINHD1X5SQUARE
- R4: value 470 -> 1K
- R7: value 10K -> 1 K
- RFM69: value RFM69 -> RFM69W; device LowPowerLab:RFM69 -> RemoteHome:RFM69W
Connections:
- net N$10 renamed S
- new net N$10: R6.1, U$5.TX
- new net N$11: R7.1, U$5.RX
- net 5V: now also C3.1; no longer JP2.1
- net A0: no longer JP2.4, R5.2
- net A1: no longer JP2.5, R7.2
- net D0_RX: now also R6.2
- net D1_TX: now also R7.2
- net D2: now also U$5.EN
- net D3: no longer JP2.2, R3.2
- net D9: no longer R14.2, R4.1
- net GND: now also C3.2, C4.2, R4.1, U$5.GND, U$5.GPIO15; no longer JP2.3, R14.1, R3.1, R5.1, R7.1
- net VCC: now also C4.1, U$5.VDD
Other:
- moved on the sheet: C1, C5, R2, R4, R7
