File: SimpleSwitchPirLightCO2_ESP03.sch (EAGLE design)
At the start: 56 parts, among them IC3 MC33269ST-3.3T3, K1 FRS1B, K2 FRS1B, K3 FRS1B, Q1 BC327SMD, T1 BC846, T2 BC846, T3 BC846, T4 BC846, X1 16 MHz

Commit message: bugfix
Parts:
- removed R10: 100, resistor:R-EU_R2512W
- removed RFM69: RFM69-ESP03, RemoteHome:RFM69-ESP03
- removed U$1: RFM12B_ANTENNA, LowPowerLab:RFM12B_ANTENNA
- added C12: 500uF, resistor:CPOL-EUSMCD
- added C4: 3,3uF, resistor:CPOL-EUE5-10.5
- added L2: 1mH, inductors:BL02RN1
- added U$5: ESP03, RemoteHome:ESP03
- C9: value 100uF -> 500uF; device resistor:CPOL-EUSMCB -> resistor:CPOL-EUSMCD
- R17, R18: value 1k -> 1 K; device resistor:R-EU_R2012 -> resistor:R-EU_M2012
Connections:
- removed net N$3: RFM69.ANT, U$1.1
- net D10_SS: no longer RFM69.SEL
- net D11_MOSI: no longer RFM69.MOSI
- net D12_MISO: no longer RFM69.MISO
- net D13_SCK: no longer RFM69.SCK
- net D2: now also U$5.EN; no longer RFM69.DIO0
- net D9: no longer RFM69.WIFI_EN
- net GND: now also C12.-, C4.-, U$5.GND, U$5.GPIO15; no longer RFM69.GND, RFM69.WIFI_GND, RFM69.WIFI_GND1
- net N$13: now also C4.+, L2.2; no longer R10.2
- net N$14: now also L2.1; no longer R10.1
- net N$28: now also U$5.TX; no longer RFM69.WIFI_TX
- net N$29: now also U$5.RX; no longer RFM69.WIFI_RX
- net VCC: now also C12.+, U$5.VDD; no longer RFM69.VCC, RFM69.WIFI_VDD
Other:
- moved on the sheet: B2, C6, R11, R17, R18, R5, R6
