File: sensorCR123.sch (EAGLE design)
At the start: 20 parts, among them IC1 LM75AD, IC4 RFM69, X1 16 MHz

Commit message: aaa
aaa
Parts:
- removed IC4: RFM69, LowPowerLab:RFM69
- added C3: 100nF, resistor:C-EUC2012
- added JP4, JP5, JP6: (no value), pinhead-2:PINHD-1X01_2.54
- added R6, R7: 1 K, resistor:R-EU_M2012
- added U$4: RFM69W, RemoteHome:RFM69W
- added U$5: ESP03, RemoteHome:ESP03
- added U1: MMA8452Q, SparkFun-Sensors:MMA8452Q
- added U2: BMP180, SparkFun-Sensors:BMP180
- JP1: device pinhead-2:PINHD-1X03_2.54-S -> pinhead-2:PINHD-1X04_2.54-S
Connections:
- new net N$10: R6.1, U$5.TX
- new net N$11: R7.1, U$5.RX
- new net N$2: C3.1, U1.BYP
- net A3: now also JP4.1
- net A4_SDA: now also U1.SDA, U2.SDA
- net A5_SCL: now also U1.SCL, U2.SCL
- net D0_RX: now also R6.2
- net D10_SS: now also U$4.SEL; no longer IC4.SEL
- net D11_MOSI: now also U$4.MOSI; no longer IC4.MOSI
- net D12_MISO: now also U$4.MISO; no longer IC4.MISO
- net D13_SCK: now also U$4.SCK; no longer IC4.SCK
- net D1_TX: now also R7.2
- net D2: now also U$4.DIO0, U$5.EN; no longer IC4.DIO0
- net D3: now also JP1.3, R4.1, U1.INT2; no longer JP1.2, R4.2
- net D4: now also JP1.4, R4.2, U1.INT1
- net D5: now also R5.1
- net D6: now also U1.VDD, U1.VDDIO, U2.VDD, U2.VDDIO
- net D7: now also JP5.1
- net D8: now also JP6.1
- net GND: now also C3.2, JP1.2, U$4.GND, U$5.GND, U$5.GPIO15, U1.GND@0, U1.GND@1, U1.GND@2, U1.SA0, U2.GND; no longer IC4.GND, R4.1, R5.1
- net N$3: now also U$4.ANT; no longer IC4.ANT
- net VCC: now also U$4.VCC, U$5.VDD; no longer IC4.VCC, JP1.3
Other:
- moved on the sheet: JP2, R4, R5

Commit message: bugfix
Parts:
- added D1: (no value), diode:DIODE-DO214BA
- added LED: L_AMBER, MySMD:LED0805
- added R8: 220, resistor:R-EU_M2012
Connections:
- new net N$4: LED.AN, R8.2
- new net N$5: D1.A, U$3.+
- net D13_SCK: now also R8.1
- net GND: now also LED.CA
- net VCC: now also D1.C; no longer U$3.+
Other:
- moved on the sheet: U$3
Changed lines of the file:
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@@
 <layer number="97" name="Info" color="7" fill="1" visible="yes" active="yes"/>
 <layer number="98" name="Guide" color="6" fill="1" visible="yes" active="yes"/>
+<layer number="99" name="SpiceOrder" color="5" fill="1" visible="yes" active="yes"/>
 <layer number="100" name="Muster" color="7" fill="1" visible="no" active="no"/>
 <layer number="101" name="Patch_Top" color="12" fill="4" visible="no" active="yes"/>
@@
 <part name="U$5" library="RemoteHome" deviceset="ESP03" device=""/>
 <part name="SUPPLY18" library="supply2" deviceset="GND" device=""/>
+<part name="LED" library="MySMD" deviceset="LED0805" device="" value="L_AMBER"/>
+<part name="R8" library="resistor" deviceset="R-EU_" device="M2012" value="220"/>
+<part name="SUPPLY19" library="supply2" deviceset="GND" device=""/>
+<part name="D1" library="diode" deviceset="DIODE-" device="DO214BA"/>
 </parts>
 <sheets>
@@
 <instance part="JP2" gate="A" x="60.96" y="160.02"/>
 <instance part="JP3" gate="A" x="124.46" y="45.72"/>
-<instance part="U$3" gate="G$1" x="109.22" y="48.26" rot="R90"/>
+<instance part="U$3" gate="G$1" x="109.22" y="43.18" rot="R90"/>
 <instance part="U1" gate="G$1" x="167.64" y="81.28"/>
 <instance part="SUPPLY10" gate="GND" x="152.4" y="60.96"/>
@@
 <instance part="U$5" gate="G$1" x="-35.56" y="40.64"/>
 <instance part="SUPPLY18" gate="GND" x="-17.78" y="35.56"/>
+<instance part="LED" gate="G$1" x="68.58" y="55.88" rot="R270"/>
+<instance part="R8" gate="G$1" x="68.58" y="68.58" rot="R270"/>
+<instance part="SUPPLY19" gate="GND" x="68.58" y="48.26"/>
+<instance part="D1" gate="G$1" x="109.22" y="55.88" rot="R90"/>
 </instances>
 <busses>
@@
 <wire x1="121.92" y1="30.48" x2="116.84" y2="30.48" width="0.1524" layer="91"/>
 <pinref part="U$3" gate="G$1" pin="-"/>
-<wire x1="109.22" y1="40.64" x2="109.22" y2="30.48" width="0.1524" layer="91"/>
+<wire x1="109.22" y1="35.56" x2="109.22" y2="30.48" width="0.1524" layer="91"/>
 <junction x="109.22" y="30.48"/>
 </segment>
@@
 <junction x="-17.78" y="38.1"/>
 </segment>
+<segment>
+<pinref part="LED" gate="G$1" pin="CA"/>
+<junction x="68.58" y="50.8"/>
+<pinref part="SUPPLY19" gate="GND" pin="GND"/>
+</segment>
 </net>
 <net name="VCC" class="0">
@@
 <pinref part="SUPPLY1" gate="1" pin="VCC"/>
 <wire x1="93.98" y1="63.5" x2="109.22" y2="63.5" width="0.1524" layer="91"/>
-<pinref part="U$3" gate="G$1" pin="+"/>
-<wire x1="109.22" y1="63.5" x2="116.84" y2="63.5" width="0.1524" layer="91"/>
 <wire x1="116.84" y1="63.5" x2="109.22" y2="63.5" width="0.1524" layer="91"/>
-<wire x1="109.22" y1="63.5" x2="109.22" y2="55.88" width="0.1524" layer="91"/>
 <junction x="109.22" y="63.5"/>
 <junction x="116.84" y="63.5"/>
 <junction x="93.98" y="63.5"/>
+<pinref part="D1" gate="G$1" pin="C"/>
+<wire x1="109.22" y1="63.5" x2="109.22" y2="58.42" width="0.1524" layer="91"/>
 </segment>
 <segment>
@@
 <label x="58.42" y="78.74" size="1.778" layer="95"/>
 <pinref part="ATMEGA328" gate="G$1" pin="PB5(SCK)"/>
+<pinref part="R8" gate="G$1" pin="1"/>
+<wire x1="68.58" y1="73.66" x2="68.58" y2="78.74" width="0.1524" layer="91"/>
+<junction x="68.58" y="78.74"/>
 </segment>
 <segment>
@@
 </segment>
 </net>
+<net name="N$4" class="0">
+<segment>
+<pinref part="R8" gate="G$1" pin="2"/>
+<pinref part="LED" gate="G$1" pin="AN"/>
+</segment>
+</net>
+<net name="N$5" class="0">
+<segment>
+<pinref part="U$3" gate="G$1" pin="+"/>
+<pinref part="D1" gate="G$1" pin="A"/>
+<wire x1="109.22" y1="50.8" x2="109.22" y2="53.34" width="0.1524" layer="91"/>
+</segment>
+</net>
